File: PCB Design/RGW LED board/RGW LED board.kicad_pcb (KiCad board)
At the start: 2 copper layers, 151.1 x 24.1 mm, 15 parts, among them J1 - R strip +, J10 - G strip +, J11 - W strip +, J12 - R strip +, J13 - G strip +, J2 - G strip +, J3 - R from above +, J4 - W strip +, J5 - G from above +, J6 - W from above +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

Commit message: Version 3 Assembly Edits
Parts:
- moved G*** 2.03 mm to (80.0, 33.0)
- moved G*** 0.76 mm to (118.1, 32.5)
Routing:
- net (no net): track 12.7 -> 0.00 mm
Other:
- board text added: "Green"
- board text added: "OJB"
- board text added: "Red"
- board text added: "White"
Changed lines of the file:
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@@
       (drillshape 0)
       (scaleselection 1)
-      (outputdirectory "../RGWGerber/")
+      (outputdirectory "../.PCBsV2/RGWGerber2/")
     )
   )
@@
   (net 6 "/W+")
   (footprint "LOGO" (layer "F.Cu")
-    (at 82.042 33.02)
+    (at 80.01 33.02)
     (attr board_only exclude_from_pos_files exclude_from_bom)
     (fp_text reference "G***" (at -0.635 -2.54) (layer "F.Fab")
@@
       (effects (font (size 1 1) (thickness 0.15)))
     )
-    (fp_text value "- G strip +" (at 2.54 5.08) (layer "F.SilkS")
+    (fp_text value "- G strip +" (at 2.54 5.715) (layer "F.SilkS")
       (effects (font (size 1 1) (thickness 0.15)))
     )
@@
       (effects (font (size 1 1) (thickness 0.15)))
     )
-    (fp_text value "- G strip +" (at 2.54 5.08) (layer "F.SilkS")
+    (fp_text value "- G strip +" (at 2.54 5.715) (layer "F.SilkS")
       (effects (font (size 1 1) (thickness 0.15)))
     )
@@
       (effects (font (size 1 1) (thickness 0.15)))
     )
-    (fp_text value "- G strip +" (at 2.54 5.08) (layer "F.SilkS")
+    (fp_text value "- G strip +" (at 2.54 5.715) (layer "F.SilkS")
       (effects (font (size 1 1) (thickness 0.15)))
     )
@@
       (effects (font (size 1 1) (thickness 0.15)))
     )
-    (fp_text value "- R strip +" (at 2.54 5.08) (layer "F.SilkS")
+    (fp_text value "- R strip +" (at 2.54 5.715) (layer "F.SilkS")
       (effects (font (size 1 1) (thickness 0.15)))
     )
@@
       (effects (font (size 1 1) (thickness 0.15)))
     )
-    (fp_text value "- R strip +" (at 2.54 5.08) (layer "F.SilkS")
+    (fp_text value "- R strip +" (at 2.54 5.715) (layer "F.SilkS")
       (effects (font (size 1 1) (thickness 0.15)))
     )
@@
   )
   (footprint "LOGO" (layer "F.Cu")
-    (at 118.872 32.512)
+    (at 118.11 32.512)
     (attr board_only exclude_from_pos_files exclude_from_bom)
     (fp_text reference "G***" (at 0 -1.905) (layer "F.Fab")
@@
       (effects (font (size 1 1) (thickness 0.15)))
     )
-    (fp_text value "- W strip +" (at 2.54 5.08) (layer "F.SilkS")
+    (fp_text value "- W strip +" (at 2.54 5.715) (layer "F.SilkS")
       (effects (font (size 1 1) (thickness 0.15)))
     )
@@
       (effects (font (size 1 1) (thickness 0.15)))
     )
-    (fp_text value "- G strip +" (at 2.54 5.08) (layer "F.SilkS")
+    (fp_text value "- G strip +" (at 2.54 5.715) (layer "F.SilkS")
       (effects (font (size 1 1) (thickness 0.15)))
     )
@@
       (effects (font (size 1 1) (thickness 0.15)))
     )
-    (fp_text value "- R strip +" (at 2.54 5.08) (layer "F.SilkS")
+    (fp_text value "- R strip +" (at 2.54 5.715) (layer "F.SilkS")
       (effects (font (size 1 1) (thickness 0.15)))
     )
@@
       (effects (font (size 1 1) (thickness 0.15)))
     )
-    (fp_text value "- W strip +" (at 2.54 5.08) (layer "F.SilkS")
+    (fp_text value "- W strip +" (at 2.54 5.715) (layer "F.SilkS")
       (effects (font (size 1 1) (thickness 0.15)))
     )
@@
       (effects (font (size 1 1) (thickness 0.15)))
     )
-    (fp_text value "- R strip +" (at 2.54 5.08) (layer "F.SilkS")
+    (fp_text value "- R strip +" (at 2.54 5.715) (layer "F.SilkS")
       (effects (font (size 1 1) (thickness 0.15)))
     )
@@
   (gr_arc (start 213.36 46.99) (mid 212.244077 49.684077) (end 209.55 50.8) (layer "Edge.Cuts") (width 0.1))
   (gr_rect (start 62.23 26.67) (end 213.36 50.8) (layer "F.Fab") (width 0.1) (fill none))
+  (gr_text "OJB" (at 154.94 32.385) (layer "F.Cu")
+    (effects (font (size 1.5 1.5) (thickness 0.3)))
+  )
   (gr_text "Made for the Rosbash Lab at Brandeis" (at 192.786 34.036) (layer "F.SilkS")
     (effects (font (size 1 1) (thickness 0.2)))
@@
     (effects (font (size 1 1) (thickness 0.2)))
   )
+  (gr_text "White\n" (at 130.175 33.02 90) (layer "F.SilkS")
+    (effects (font (size 1.5 1.5) (thickness 0.3)))
+  )
+  (gr_text "Green\n" (at 162.56 32.385 90) (layer "F.SilkS")
+    (effects (font (size 1.5 1.5) (thickness 0.3)))
+  )
+  (gr_text "Red" (at 92.71 33.02 90) (layer "F.SilkS")
+    (effects (font (size 1.5 1.5) (thickness 0.3)))
+  )
   (gr_text "Flybox RGW Board\n" (at 192.786 31.115) (layer "F.SilkS")
     (effects (font (size 2 2) (thickness 0.2)))
   )
-  (segment (start 157.48 33.02) (end 156.21 33.02) (width 0.25) (layer "F.Cu") (net 0))
-  (segment (start 156.845 32.385) (end 156.845 33.02) (width 0.25) (layer "F.Cu") (net 0))
-  (segment (start 154.305 32.385) (end 154.94 32.385) (width 0.25) (layer "F.Cu") (net 0))
-  (segment (start 156.21 32.385) (end 156.21 33.655) (width 0.25) (layer "F.Cu") (net 0))
-  (segment (start 153.67 33.02) (end 153.035 33.655) (width 0.25) (layer "F.Cu") (net 0))
-  (segment (start 152.4 33.02) (end 153.035 32.385) (width 0.25) (layer "F.Cu") (net 0))
-  (segment (start 154.305 33.655) (end 154.305 33.02) (width 0.25) (layer "F.Cu") (net 0))
-  (segment (start 156.21 33.655) (end 156.845 33.655) (width 0.25) (layer "F.Cu") (net 0))
-  (segment (start 153.035 32.385) (end 153.67 33.02) (width 0.25) (layer "F.Cu") (net 0))
-  (segment (start 156.845 33.655) (end 157.48 33.02) (width 0.25) (layer "F.Cu") (net 0))
-  (segment (start 154.94 32.385) (end 154.94 33.655) (width 0.25) (layer "F.Cu") (net 0))
-  (segment (start 156.21 32.385) (end 156.845 32.385) (width 0.25) (layer "F.Cu") (net 0))
-  (segment (start 153.035 33.655) (end 152.4 33.02) (width 0.25) (layer "F.Cu") (net 0))
-  (segment (start 154.94 33.655) (end 154.305 33.655) (width 0.25) (layer "F.Cu") (net 0))
-  (segment (start 154.94 32.385) (end 155.575 32.385) (width 0.25) (layer "F.Cu") (net 0))
   (via (at 66.04 30.48) (size 5) (drill 3.4) (layers "F.Cu" "B.Cu") (free) (net 0))
   (via (at 209.55 30.48) (size 5) (drill 3.4) (layers "F.Cu" "B.Cu") (free) (net 0))
@@
   (segment (start 168.656 40.287) (end 168.656 40.132) (width 0.635) (layer "B.Cu") (net 4))
   (segment (start 168.656 40.132) (end 165.1 36.576) (width 0.635) (layer "B.Cu") (net 4))
-  (segment (start 139.192 36.83) (end 139.065 36.83) (width 0.635) (layer "F.Cu") (net 5))
+  (segment (start 140.335 38.1) (end 135.255 33.02) (width 0.635) (layer "F.Cu") (net 5))
   (segment (start 141.732 39.37) (end 174.625 39.37) (width 0.635) (layer "F.Cu") (net 5))
   (segment (start 130.429 37.846) (end 95.504 37.846) (width 0.635) (layer "F.Cu") (net 5))
   (segment (start 92.71 40.64) (end 92.71 42.545) (width 0.635) (layer "F.Cu") (net 5))
   (segment (start 174.625 39.37) (end 177.8 42.545) (width 0.635) (layer "F.Cu") (net 5))
-  (segment (start 139.065 36.83) (end 135.255 33.02) (width 0.635) (layer "F.Cu") (net 5))
   (segment (start 135.255 33.02) (end 130.429 37.846) (width 0.635) (layer "F.Cu") (net 5))
   (segment (start 95.504 37.846) (end 92.71 40.64) (width 0.635) (layer "F.Cu") (net 5))
-  (via (at 139.192 36.83) (size 0.8) (drill 0.4) (layers "F.Cu" "B.Cu") (free) (net 5))
+  (via (at 140.335 38.1) (size 0.8) (drill 0.4) (layers "F.Cu" "B.Cu") (free) (net 5))
   (via (at 141.732 39.37) (size 0.8) (drill 0.4) (layers "F.Cu" "B.Cu") (free) (net 5))
-  (segment (start 139.192 36.83) (end 141.732 39.37) (width 0.635) (layer "B.Cu") (net 5))
+  (segment (start 140.462 38.1) (end 141.732 39.37) (width 0.635) (layer "B.Cu") (net 5))
+  (segment (start 140.335 38.1) (end 140.462 38.1) (width 0.635) (layer "B.Cu") (net 5))
+  (segment (start 97.79 40.64) (end 99.2155 39.2145) (width 0.635) (layer "F.Cu") (net 6))
+  (segment (start 99.2155 39.2145) (end 112.648041 39.2145) (width 0.635) (layer "F.Cu") (net 6))
   (segment (start 145.415 38.1) (end 140.335 33.02) (width 0.635) (layer "F.Cu") (net 6))
-  (segment (start 138.43 38.1) (end 144.78 38.1) (width 0.635) (layer "F.Cu") (net 6))
   (segment (start 144.78 38.1) (end 145.415 38.1) (width 0.635) (layer "F.Cu") (net 6))
-  (segment (start 99.495 38.935) (end 137.595 38.935) (width 0.635) (layer "F.Cu") (net 6))
-  (segment (start 97.79 40.64) (end 99.495 38.935) (width 0.635) (layer "F.Cu") (net 6))
+  (segment (start 140.434459 39.37) (end 141.704459 38.1) (width 0.635) (layer "F.Cu") (net 6))
   (segment (start 144.78 38.1) (end 178.435 38.1) (width 0.635) (layer "F.Cu") (net 6))
-  (segment (start 138.43 38.1) (end 137.595 38.935) (width 0.635) (layer "F.Cu") (net 6))
-  (segment (start 178.435 38.1) (end 182.88 42.545) (width 0.635) (layer "F.Cu") (net 6))
   (segment (start 97.79 42.545) (end 97.79 40.64) (width 0.635) (layer "F.Cu") (net 6))
+  (segment (start 112.648041 39.2145) (end 112.803541 39.37) (width 0.635) (layer "F.Cu") (net 6))
+  (segment (start 112.803541 39.37) (end 140.434459 39.37) (width 0.635) (layer "F.Cu") (net 6))
+  (segment (start 141.704459 38.1) (end 144.78 38.1) (width 0.635) (layer "F.Cu") (net 6))
+  (segment (start 178.435 38.1) (end 182.88 42.545) (width 0.635) (layer "F.Cu") (net 6))
   (group "" (id 0aaa3c9e-91d2-41d7-9fff-f8e391e88df2)
     (members
