File: PCB Design/RGW LED board/RGW LED board.kicad_pcb (KiCad board)
At the start: 2 copper layers, 151.1 x 24.1 mm, 15 parts, among them J1 - R strip +, J10 - G strip +, J11 - W strip +, J12 - R strip +, J13 - G strip +, J2 - G strip +, J3 - R from above +, J4 - W strip +, J5 - G from above +, J6 - W from above +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

Commit message: Fixed capitalization
Other:
- board text added: "FlyBox RGW Board"
- board text removed: "Flybox RGW Board"
Changed lines of the file:
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@@
     (effects (font (size 1.5 1.5) (thickness 0.3)))
   )
-  (gr_text "Flybox RGW Board\n" (at 192.786 31.115) (layer "F.SilkS")
+  (gr_text "FlyBox RGW Board\n" (at 192.786 31.115) (layer "F.SilkS")
     (effects (font (size 2 2) (thickness 0.2)))
   )
