File: PCB Design/IR FANS LED board/IR FANS LED board.kicad_pcb (KiCad board)
At the start: 2 copper layers, 148.6 x 29.2 mm, 11 parts, among them J1 Fan, J2 Fan, J3 IR, J4 Fans from above, J5 IR, J6 IR from above, J7 IR, J8 Fan, J9 Fan

Commit message: Version 3 Assembly Edits
Parts:
- moved J6 5.46 mm to (163.2, 27.3), turned to 180 degrees
- moved J4 3.18 mm to (188.0, 27.3)
- moved J3 0.63 mm to (131.4, 40.0)
- moved J5 0.63 mm to (166.4, 40.0)
- moved J7 0.63 mm to (100.3, 40.0)
Routing:
- net /IR LED-: track 85.6 -> 103.2 mm
- net (no net): track 12.7 -> 0.00 mm
- net /IR LED+: track 87.9 -> 95.7 mm
- net /HV5: track 187.5 -> 189.6 mm
- net /12V: track 166.8 -> 165.5 mm
- net /GND: track 235.6 -> 236.8 mm
- net /X: track 178.6 -> 179.5 mm
Other:
- board text added: "GND 12V RPM Signal PWM Signal"
- board text added: "OJB"
- board text added: "PWM Signal RPM Signal 12V GND"
- board text removed: "GND-black 12V-yellow Signal-blue"
- board text removed: "Signal-blue 12V-yellow GND-black"

Commit message: Fixed capitalization
Other:
- board text added: "FlyBox IR and Fans Board"
- board text removed: "Flybox IR and Fans Board"
Changed lines of the file:
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@@
     (effects (font (size 0.8 0.6) (thickness 0.125)) (justify left))
   )
-  (gr_text "Flybox IR and Fans Board\n" (at 127.762 24.638) (layer "F.SilkS")
+  (gr_text "FlyBox IR and Fans Board\n" (at 127.762 24.638) (layer "F.SilkS")
     (effects (font (size 2 2) (thickness 0.2)))
   )

Commit message: Zachary final review of PCBs
Changed lines of the file:
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@@
   (setup
     (pad_to_mask_clearance 0)
-    (grid_origin 172.72 30.48)
+    (grid_origin 54.356 51.816)
     (pcbplotparams
       (layerselection 0x00010fc_ffffffff)
@@
   (gr_line (start 204.47 17.78) (end 63.5 17.78) (layer "Edge.Cuts") (width 0.1))
   (gr_rect (start 59.69 17.78) (end 208.28 46.99) (layer "F.Fab") (width 0.1) (fill none))
-  (gr_text "OJB" (at 183.515 39.37) (layer "F.Cu")
+  (gr_text "OJB" (at 183.642 41.402) (layer "F.Cu")
     (effects (font (size 1.5 1.5) (thickness 0.3)))
   )
